Commit message: Cleaned up pipette driver, pipette description, pipette moveit config and updated readme. Using a cylinder for Mesh for now

File: src/custom-ur-descriptions/pipette_description/urdf/pipette.urdf.xacro (robot description, xacro)
@@ -2,9 +2,4 @@
 <robot xmlns:xacro="http://ros.org/wiki/xacro" name="pipette">
   <xacro:arg name="parent" default="tool0"/>
-  <xacro:arg name="serial_port" default="/dev/ttyUSB0"/>
-  <xacro:arg name="baudrate" default="115200"/>
-  <xacro:arg name="plunger_max" default="1.0"/>
-  <xacro:arg name="tip_eject_max" default="1.0"/>
-  <xacro:arg name="use_fake_hardware" default="true"/>
   <xacro:include filename="$(find pipette_description)/urdf/pipette_macro.urdf.xacro"/>
   <link name="$(arg parent)"/>
@@ -13,9 +8,4 @@
     prefix=""
     parent="$(arg parent)"
-    serial_port="$(arg serial_port)"
-    baudrate="$(arg baudrate)"
-    plunger_max="$(arg plunger_max)"
-    tip_eject_max="$(arg tip_eject_max)"
-    use_fake_hardware="$(arg use_fake_hardware)"
   />
 </robot>

File: src/custom-ur-descriptions/pipette_description/urdf/pipette_macro.urdf.xacro (robot description, xacro)
@@ -2,8 +2,7 @@
 <robot xmlns:xacro="http://ros.org/wiki/xacro">
   <!--
-    Static URDF description for pipette tool with ros2_control integration
+    Static URDF description for pipette tool
     Replace placeholder meshes with your actual CAD files
   -->
-  <xacro:include filename="$(find pipette_description)/urdf/pipette.ros2_control.xacro"/>
   <xacro:macro
     name="pipette"
@@ -11,23 +10,8 @@
             prefix
             parent
-            serial_port
-            baudrate
-            plunger_max
-            tip_eject_max
-            use_fake_hardware
             pipette_mass:=0.200
             xyz:='0 0 0'
             rpy:='0 0 0'"
   >
-    <!-- ros2_control parameters -->
-    <xacro:pipette_ros2_control
-      name="${name}"
-      prefix="${prefix}"
-      serial_port="${serial_port}"
-      baudrate="${baudrate}"
-      plunger_max="${plunger_max}"
-      tip_eject_max="${tip_eject_max}"
-      use_fake_hardware="${use_fake_hardware}"
-    />
     <!-- Pipette physical dimensions (adjust based on your CAD) -->
     <xacro:property name="pipette_length" value="0.15"/>  <!-- 15cm length -->
@@ -95,5 +79,5 @@
       <child link="${prefix}plunger_link"/>
       <axis xyz="0 0 1"/>  <!-- Z-axis movement (up/down) -->
-      <limit effort="10.0" lower="0.0" upper="${plunger_max}" velocity="0.01"/>
+      <limit effort="10.0" lower="0.0" upper="1.0" velocity="0.1"/>
     </joint>
     <link name="${prefix}plunger_link">
@@ -112,5 +96,5 @@
       <child link="${prefix}tip_eject_link"/>
       <axis xyz="0 0 1"/>  <!-- Z-axis movement (up/down) -->
-      <limit effort="5.0" lower="0.0" upper="${tip_eject_max}" velocity="0.01"/>
+      <limit effort="5.0" lower="0.0" upper="1.0" velocity="0.1"/>
     </joint>
     <link name="${prefix}tip_eject_link">
@@ -124,5 +108,5 @@
     <!-- Tool tip reference frame -->
     <joint name="${prefix}pipette_tip_joint" type="fixed">
-      <origin xyz="0 0 ${pipette_length + 0.01}" rpy="0 0 0"/>
+      <origin xyz="0 0 ${pipette_length}" rpy="0 0 0"/>
       <parent link="${prefix}pipette_base_link"/>
       <child link="${prefix}pipette_tip_link"/>
