Commit message: Finished pipette description. Updated the cylinder to actual mesh

File: src/custom-ur-descriptions/pipette_description/urdf/pipette_macro.urdf.xacro (robot description, xacro)
@@ -15,6 +15,34 @@
   >
     <!-- Pipette physical dimensions (adjust based on your CAD) -->
-    <xacro:property name="pipette_length" value="0.15"/>  <!-- 15cm length -->
+    <xacro:property name="pipette_length" value="0.34"/>  <!-- 15cm length -->
     <xacro:property name="pipette_radius" value="0.02"/>   <!-- 2cm radius -->
+    <!-- Base position and orientation for all components -->
+    <xacro:property name="base_xyz_x" value="-0.0860"/>
+    <xacro:property name="base_xyz_y" value="-0.3224"/>
+    <xacro:property name="base_xyz_z" value="-0.058"/>
+    <xacro:property name="base_rpy_x" value="0"/>
+    <xacro:property name="base_rpy_y" value="0"/>
+    <xacro:property name="base_rpy_z" value="0"/>
+    <!-- Visual component offsets -->
+    <xacro:property name="visual_xyz_offset_x" value="0"/>
+    <xacro:property name="visual_xyz_offset_y" value="0.0043"/>
+    <xacro:property name="visual_xyz_offset_z" value="0.0183" />
+    <xacro:property name="visual_rpy_offset_x" value="0"/>
+    <xacro:property name="visual_rpy_offset_y" value="0"/>
+    <xacro:property name="visual_rpy_offset_z" value="0"/>
+    <!-- Collision component offsets -->
+    <xacro:property name="collision_xyz_offset_x" value="0"/>
+    <xacro:property name="collision_xyz_offset_y" value="0"/>
+    <xacro:property name="collision_xyz_offset_z" value="0"/>
+    <xacro:property name="collision_rpy_offset_x" value="0"/>
+    <xacro:property name="collision_rpy_offset_y" value="0"/>
+    <xacro:property name="collision_rpy_offset_z" value="0"/>
+    <!-- Inertial component offsets -->
+    <xacro:property name="inertial_xyz_offset_x" value="0"/>
+    <xacro:property name="inertial_xyz_offset_y" value="0"/>
+    <xacro:property name="inertial_xyz_offset_z" value="0"/>
+    <xacro:property name="inertial_rpy_offset_x" value="0"/>
+    <xacro:property name="inertial_rpy_offset_y" value="0"/>
+    <xacro:property name="inertial_rpy_offset_z" value="0"/>
     <!-- Main attachment joint -->
     <joint name="${prefix}pipette_attachment_joint" type="fixed">
@@ -23,12 +51,21 @@
       <child link="${prefix}pipette_base_link"/>
     </joint>
-    <!-- Main pipette body -->
-    <link name="${prefix}pipette_base_link">
+    <!-- Main pipette body (base positioning) -->
+    <link name="${prefix}pipette_base_link"/>
+    <!-- Intermediate joint for 90-degree rotation -->
+    <joint name="${prefix}pipette_orientation_joint" type="fixed">
+      <origin xyz="-0.09 -0.055 ${pipette_length}" rpy="${base_rpy_x - 1.5708} ${base_rpy_y} ${base_rpy_z}"/>
+      <parent link="${prefix}pipette_base_link"/>
+      <child link="${prefix}pipette_body_link"/>
+    </joint>
+    <!-- Pipette body link with visual, collision and inertial -->
+    <link name="${prefix}pipette_body_link">
       <visual>
-        <origin xyz="0 0 ${pipette_length/2}" rpy="0 0 0"/>
+        <origin xyz="${visual_xyz_offset_x} ${visual_xyz_offset_y} ${visual_xyz_offset_z}"
+                rpy="${visual_rpy_offset_x} ${visual_rpy_offset_y} ${visual_rpy_offset_z}"/>
         <geometry>
           <!-- Replace this cylinder with your CAD mesh -->
-          <!-- <mesh filename="package://pipette_description/meshes/visual/pipette_body.dae"/> -->
-          <cylinder length="${pipette_length}" radius="${pipette_radius}"/>
+          <mesh filename="package://pipette_description/meshes/visual/pipettor_visual.stl" scale="0.001 0.001 0.001" />
+          <!-- <cylinder length="${pipette_length}" radius="${pipette_radius}"/> -->
         </geometry>
         <material name="pipette_gray">
@@ -37,13 +74,15 @@
       </visual>
       <collision>
-        <origin xyz="0 0 ${pipette_length/2}" rpy="0 0 0"/>
+        <origin xyz="${collision_xyz_offset_x} ${collision_xyz_offset_y} ${collision_xyz_offset_z}"
+                rpy="${collision_rpy_offset_x} ${collision_rpy_offset_y} ${collision_rpy_offset_z}"/>
         <geometry>
           <!-- Replace this cylinder with simplified collision mesh -->
-          <!-- <mesh filename="package://pipette_description/meshes/collision/pipette_body.stl"/> -->
-          <cylinder length="${pipette_length}" radius="${pipette_radius}"/>
+          <mesh filename="package://pipette_description/meshes/collision/pipettor_collision.stl" scale="0.001 0.001 0.001" />
+          <!-- <cylinder length="${pipette_length}" radius="${pipette_radius}"/> -->
         </geometry>
       </collision>
       <inertial>
-        <origin xyz="0 0 ${pipette_length/2}" rpy="0 0 0"/>
+        <origin xyz="${inertial_xyz_offset_x} ${inertial_xyz_offset_y} ${inertial_xyz_offset_z}"
+                rpy="${inertial_rpy_offset_x} ${inertial_rpy_offset_y} ${inertial_rpy_offset_z}"/>
         <mass value="${pipette_mass}"/>
         <inertia ixx="${pipette_mass * (3 * pipette_radius * pipette_radius + pipette_length * pipette_length) / 12}"
@@ -72,38 +111,6 @@
       </visual>
     </link>
-    <!-- Conceptual plunger link for ros2_control (no visual representation) -->
-    <!-- This represents the internal plunger mechanism -->
-    <joint name="${prefix}plunger_joint" type="prismatic">
-      <origin xyz="0 0 ${pipette_length}" rpy="0 0 0"/>
-      <parent link="${prefix}pipette_base_link"/>
-      <child link="${prefix}plunger_link"/>
-      <axis xyz="0 0 1"/>  <!-- Z-axis movement (up/down) -->
-      <limit effort="10.0" lower="0.0" upper="1.0" velocity="0.1"/>
-    </joint>
-    <link name="${prefix}plunger_link">
-      <!-- No visual/collision geometry - this is handled by hardware interface -->
-      <inertial>
-        <origin xyz="0 0 0" rpy="0 0 0"/>
-        <mass value="0.001"/>  <!-- Minimal mass -->
-        <inertia ixx="1E-9" ixy="0.0" ixz="0.0" iyy="1E-9" iyz="0.0" izz="1E-9"/>
-      </inertial>
-    </link>
-    <!-- Conceptual tip ejection link for ros2_control (no visual representation) -->
-    <!-- This represents the tip ejection mechanism -->
-    <joint name="${prefix}tip_eject_joint" type="prismatic">
-      <origin xyz="0 0 ${pipette_length}" rpy="0 0 0"/>
-      <parent link="${prefix}pipette_base_link"/>
-      <child link="${prefix}tip_eject_link"/>
-      <axis xyz="0 0 1"/>  <!-- Z-axis movement (up/down) -->
-      <limit effort="5.0" lower="0.0" upper="1.0" velocity="0.1"/>
-    </joint>
-    <link name="${prefix}tip_eject_link">
-      <!-- No visual/collision geometry - this is handled by hardware interface -->
-      <inertial>
-        <origin xyz="0 0 0" rpy="0 0 0"/>
-        <mass value="0.001"/>  <!-- Minimal mass -->
-        <inertia ixx="1E-9" ixy="0.0" ixz="0.0" iyy="1E-9" iyz="0.0" izz="1E-9"/>
-      </inertial>
-    </link>
+    <!-- Plunger and tip ejection are handled by external driver -->
+    <!-- No joints needed - pipette control is managed outside of MoveIt -->
     <!-- Tool tip reference frame -->
     <joint name="${prefix}pipette_tip_joint" type="fixed">

File: src/custom-ur-descriptions/ur5e_pipette_robot_description/urdf/ur_with_pipette.xacro (robot description, xacro)
@@ -95,18 +95,13 @@
    </xacro:ur_robot>
   <!-- pipette tool -->
-    <xacro:arg name="serial_port" default="/tmp/ttyUR"/>
-    <xacro:arg name="baudrate" default="115200"/>
-    <xacro:arg name="plunger_max" default="0.010"/>
-    <xacro:arg name="tip_eject_max" default="0.005"/>
+    <xacro:arg name="pipette_mass" default="0.200"/>
+    <xacro:arg name="pipette_xyz" default="0 0 0"/>
+    <xacro:arg name="pipette_rpy" default="0 0 0"/>
     <xacro:pipette
       name="pipette"
       prefix="$(arg tf_prefix)"
-      parent="$(arg tf_prefix)flange"
-      serial_port="$(arg serial_port)"
-      baudrate="$(arg baudrate)"
-      plunger_max="$(arg plunger_max)"
-      tip_eject_max="$(arg tip_eject_max)"
-      use_fake_hardware="$(arg mock_hardware)"
-      xyz="0 0 0"
-      rpy="0 0 0"/>
+      parent="$(arg tf_prefix)tool0"
+      pipette_mass="$(arg pipette_mass)"
+      xyz="$(arg pipette_xyz)"
+      rpy="$(arg pipette_rpy)"/>
 </robot>
